Commit message: Fix non-fixed joint error and corrected orientation of wheels

File: vector_description/urdf/robot.urdf.xacro (robot description, xacro)
@@ -3,5 +3,5 @@
   <!-- Xacro Properties -->
   <!-- Mathematical constant -->
-  <xacro:property name="pi1" value="3.14159"/>
+  <!-- <xacro:property name="pi" value="3.14159"/> -->
   <!-- Base dimensions -->
   <xacro:property name="base_length" value="0.5"/>         <!-- Length of the base -->
@@ -9,5 +9,5 @@
   <xacro:property name="base_height" value="0.2"/>         <!-- Height of the base -->
   <xacro:property name="base_ground_clearance" value="0.1"/> <!-- Distance from ground to base bottom -->
-  <!-- Wheel placement (assumed symmetric) -->
+  <!-- Wheel placement (symmetric) -->
   <xacro:property name="wheel_base" value="0.4"/>          <!-- Distance between front and back wheels -->
   <xacro:property name="wheel_track" value="0.3"/>         <!-- Distance between left and right wheels -->
@@ -19,5 +19,5 @@
     <inertial>
       <!-- Orientation may be adjusted based on your modeling convention -->
-      <origin xyz="0 0 0" rpy="${pi1/2} 0 ${pi1/2}"/>
+      <origin xyz="0 0 0" rpy="${pi/2} 0 ${pi/2}"/>
       <mass value="${m}"/>
       <inertia ixx="${(m/12) * (h*h + d*d)}" ixy="0.0" ixz="0.0"
@@ -28,5 +28,5 @@
   <xacro:macro name="cylinder_inertia" params="m r h">
     <inertial>
-      <origin xyz="0 0 0" rpy="${pi1/2} 0 0"/>
+      <origin xyz="0 0 0" rpy="${pi/2} 0 0"/>
       <mass value="${m}"/>
       <inertia ixx="${(m/12) * (3*r*r + h*h)}" ixy="0" ixz="0"
@@ -63,9 +63,9 @@
        z_offset is set so that the wheel center is at the ground level (z = wheel_radius).
   -->
-  <xacro:macro name="wheel" params="name x_offset y_offset z_offset">
+  <xacro:macro name="wheel" params="name x_offset y_offset z_offset is_right">
     <link name="${name}">
       <visual>
         <!-- Rotate the cylinder so its axis (default along z) aligns with the desired rolling axis -->
-        <origin xyz="0 0 0" rpy="0 1.5708 0"/>
+        <origin xyz="0 0 0" rpy="0 0 ${pi/2}"/>
         <geometry>
           <cylinder radius="${wheel_radius}" length="${wheel_thickness}"/>
@@ -84,10 +84,15 @@
       <xacro:cylinder_inertia m="1" r="${wheel_radius}" h="${wheel_thickness}"/>
     </link>
-    <joint name="${name}_joint" type="fixed">
+    <joint name="${name}_joint" type="continuous">
       <parent link="base_link"/>
       <child link="${name}"/>
-      <origin xyz="${x_offset} ${y_offset} ${z_offset}" rpy="${pi1/2} 0 0"/>
+      <xacro:if value="${is_right}">
+        <origin xyz="${x_offset} ${y_offset} ${z_offset}" rpy="${pi/2} 0 0"/>
+      </xacro:if>
+      <xacro:unless value="${is_right}">
+        <origin xyz="${x_offset} ${y_offset} ${z_offset}" rpy="${-pi/2} 0 ${0}"/>
+      </xacro:unless>
       <!-- Set the axis to align with the rolling direction; adjust if needed -->
-      <axis xyz="1 0 0"/>
+      <axis xyz="0 0 1"/>
       <limit effort="5.0" velocity="5.0"/>
     </joint>
@@ -97,7 +102,7 @@
   <!-- Left wheels: y_offset = +wheel_track/2, Right wheels: y_offset = -wheel_track/2 -->
   <!-- z_offset is set to wheel_radius so that the wheel touches the ground -->
-  <xacro:wheel name="front_left_wheel"  x_offset="${wheel_base/2}"  y_offset="${wheel_track/2}"  z_offset="${wheel_radius}"/>
-  <xacro:wheel name="front_right_wheel" x_offset="${wheel_base/2}"  y_offset="${-wheel_track/2}" z_offset="${wheel_radius}"/>
-  <xacro:wheel name="rear_left_wheel"   x_offset="${-wheel_base/2}" y_offset="${wheel_track/2}"  z_offset="${wheel_radius}"/>
-  <xacro:wheel name="rear_right_wheel"  x_offset="${-wheel_base/2}" y_offset="${-wheel_track/2}" z_offset="${wheel_radius}"/>
+  <xacro:wheel name="front_left_wheel"  x_offset="${wheel_base/2}"  y_offset="${wheel_track/2}"  z_offset="${wheel_radius}" is_right="false"/>
+  <xacro:wheel name="front_right_wheel" x_offset="${wheel_base/2}"  y_offset="${-wheel_track/2}" z_offset="${wheel_radius}" is_right="true"/>
+  <xacro:wheel name="rear_left_wheel"   x_offset="${-wheel_base/2}" y_offset="${wheel_track/2}"  z_offset="${wheel_radius}" is_right="false"/>
+  <xacro:wheel name="rear_right_wheel"  x_offset="${-wheel_base/2}" y_offset="${-wheel_track/2}" z_offset="${wheel_radius}" is_right="true"/>
 </robot>

Commit message: Refactor URDF files to define a new robot model and include utility macros

File: vector_description/urdf/robot.urdf.xacro (robot description, xacro)
@@ -1,108 +1,7 @@
 <?xml version="1.0"?>
-<robot name="four_wheel_robot" xmlns:xacro="http://ros.org/wiki/xacro">
-  <!-- Xacro Properties -->
-  <!-- Mathematical constant -->
-  <!-- <xacro:property name="pi" value="3.14159"/> -->
-  <!-- Base dimensions -->
-  <xacro:property name="base_length" value="0.5"/>         <!-- Length of the base -->
-  <xacro:property name="base_width" value="0.3"/>          <!-- Width of the base -->
-  <xacro:property name="base_height" value="0.2"/>         <!-- Height of the base -->
-  <xacro:property name="base_ground_clearance" value="0.1"/> <!-- Distance from ground to base bottom -->
-  <!-- Wheel placement (symmetric) -->
-  <xacro:property name="wheel_base" value="0.4"/>          <!-- Distance between front and back wheels -->
-  <xacro:property name="wheel_track" value="0.3"/>         <!-- Distance between left and right wheels -->
-  <!-- Wheel dimensions -->
-  <xacro:property name="wheel_radius" value="0.1"/>
-  <xacro:property name="wheel_thickness" value="0.05"/>
-  <!-- Inertia Macros -->
-  <xacro:macro name="box_inertia" params="m w h d">
-    <inertial>
-      <!-- Orientation may be adjusted based on your modeling convention -->
-      <origin xyz="0 0 0" rpy="${pi/2} 0 ${pi/2}"/>
-      <mass value="${m}"/>
-      <inertia ixx="${(m/12) * (h*h + d*d)}" ixy="0.0" ixz="0.0"
-               iyy="${(m/12) * (w*w + d*d)}" iyz="0.0"
-               izz="${(m/12) * (w*w + h*h)}"/>
-    </inertial>
-  </xacro:macro>
-  <xacro:macro name="cylinder_inertia" params="m r h">
-    <inertial>
-      <origin xyz="0 0 0" rpy="${pi/2} 0 0"/>
-      <mass value="${m}"/>
-      <inertia ixx="${(m/12) * (3*r*r + h*h)}" ixy="0" ixz="0"
-               iyy="${(m/12) * (3*r*r + h*h)}" iyz="0"
-               izz="${(m/2) * (r*r)}"/>
-    </inertial>
-  </xacro:macro>
-  <!-- Base Link Definition -->
-  <link name="base_link">
-    <visual>
-      <!-- Raise the base so its bottom is at ground clearance -->
-      <origin xyz="0 0 ${base_ground_clearance + base_height/2}" rpy="0 0 0"/>
-      <geometry>
-        <box size="${base_length} ${base_width} ${base_height}"/>
-      </geometry>
-      <material name="blue">
-        <color rgba="0 0 1 1"/>
-      </material>
-    </visual>
-    <collision>
-      <origin xyz="0 0 ${base_ground_clearance + base_height/2}" rpy="0 0 0"/>
-      <geometry>
-        <box size="${base_length} ${base_width} ${base_height}"/>
-      </geometry>
-    </collision>
-    <!-- Use box_inertia macro for base_link (mass = 10) -->
-    <xacro:box_inertia m="10" w="${base_width}" h="${base_height}" d="${base_length}"/>
-  </link>
-  <!-- Wheel Macro -->
-  <!--
-       The macro takes a wheel name and an offset (x,y,z) relative to the base_link.
-       Here, x_offset is chosen as half the wheel_base (front wheels: +, rear: -).
-       y_offset is half the wheel_track (left: positive, right: negative).
-       z_offset is set so that the wheel center is at the ground level (z = wheel_radius).
-  -->
-  <xacro:macro name="wheel" params="name x_offset y_offset z_offset is_right">
-    <link name="${name}">
-      <visual>
-        <!-- Rotate the cylinder so its axis (default along z) aligns with the desired rolling axis -->
-        <origin xyz="0 0 0" rpy="0 0 ${pi/2}"/>
-        <geometry>
-          <cylinder radius="${wheel_radius}" length="${wheel_thickness}"/>
-        </geometry>
-        <material name="black">
-          <color rgba="0 0 0 1"/>
-        </material>
-      </visual>
-      <collision>
-        <origin xyz="0 0 0" rpy="0 1.5708 0"/>
-        <geometry>
-          <cylinder radius="${wheel_radius}" length="${wheel_thickness}"/>
-        </geometry>
-      </collision>
-      <!-- Use cylinder_inertia for the wheel (mass = 1) -->
-      <xacro:cylinder_inertia m="1" r="${wheel_radius}" h="${wheel_thickness}"/>
-    </link>
-    <joint name="${name}_joint" type="continuous">
-      <parent link="base_link"/>
-      <child link="${name}"/>
-      <xacro:if value="${is_right}">
-        <origin xyz="${x_offset} ${y_offset} ${z_offset}" rpy="${pi/2} 0 0"/>
-      </xacro:if>
-      <xacro:unless value="${is_right}">
-        <origin xyz="${x_offset} ${y_offset} ${z_offset}" rpy="${-pi/2} 0 ${0}"/>
-      </xacro:unless>
-      <!-- Set the axis to align with the rolling direction; adjust if needed -->
-      <axis xyz="0 0 1"/>
-      <limit effort="5.0" velocity="5.0"/>
-    </joint>
-  </xacro:macro>
-  <!-- Instantiate Four Wheels -->
-  <!-- Front wheels: x_offset = +wheel_base/2, Rear wheels: x_offset = -wheel_base/2 -->
-  <!-- Left wheels: y_offset = +wheel_track/2, Right wheels: y_offset = -wheel_track/2 -->
-  <!-- z_offset is set to wheel_radius so that the wheel touches the ground -->
-  <xacro:wheel name="front_left_wheel"  x_offset="${wheel_base/2}"  y_offset="${wheel_track/2}"  z_offset="${wheel_radius}" is_right="false"/>
-  <xacro:wheel name="front_right_wheel" x_offset="${wheel_base/2}"  y_offset="${-wheel_track/2}" z_offset="${wheel_radius}" is_right="true"/>
-  <xacro:wheel name="rear_left_wheel"   x_offset="${-wheel_base/2}" y_offset="${wheel_track/2}"  z_offset="${wheel_radius}" is_right="false"/>
-  <xacro:wheel name="rear_right_wheel"  x_offset="${-wheel_base/2}" y_offset="${-wheel_track/2}" z_offset="${wheel_radius}" is_right="true"/>
+<robot name="vector_robot" xmlns:xacro="http://ros.org/wiki/xacro">
+  <!-- Include utility macros and properties -->
+  <xacro:include filename="$(find vector_description)/urdf/utils.urdf.xacro" />
+  <!-- Include the model definition -->
+  <xacro:include filename="$(find vector_description)/urdf/model.urdf.xacro" />
 </robot>

File: vector_description/urdf/utils.urdf.xacro (robot description, xacro)
@@ -3,57 +3,85 @@
   <!-- Materials -->
   <material name="white">
-    <color rgba="1 1 1 1"/>
+    <color rgba="1 1 1 1" />
   </material>
   <material name="red">
-    <color rgba="1 0 0 1"/>
+    <color rgba="1 0 0 1" />
   </material>
   <material name="green">
-    <color rgba="0 1 0 1"/>
+    <color rgba="0 1 0 1" />
   </material>
   <material name="blue">
-    <color rgba="0 0 1 1"/>
+    <color rgba="0 0 1 1" />
   </material>
   <material name="yellow">
-    <color rgba="1 1 0 1"/>
+    <color rgba="1 1 0 1" />
   </material>
   <material name="black">
-    <color rgba="0 0 0 1"/>
+    <color rgba="0 0 0 1" />
   </material>
   <material name="SaxionGreen">
-    <color rgba="0 0.612 0.510 1"/>
+    <color rgba="0 0.612 0.510 1" />
   </material>
-  <!-- Inertia macros -->
+  <!-- Inertia Macros -->
   <xacro:macro name="box_inertia" params="m w h d">
     <inertial>
-      <origin xyz="0 0 0" rpy="${pi1/2} 0 ${pi1/2}"/>
-      <mass value="${m}"/>
-      <inertia ixx="${(m/12) * (h*h + d*d)}" ixy="0.0" ixz="0.0" iyy="${(m/12) * (w*w + d*d)}" iyz="0.0" izz="${(m/12) * (w*w + h*h)}"/>
+      <!-- Orientation may be adjusted based on your modeling convention -->
+      <origin xyz="0 0 0" rpy="${pi/2} 0 ${pi/2}" />
+      <mass value="${m}" />
+      <inertia ixx="${(m/12) * (h*h + d*d)}" ixy="0.0" ixz="0.0"
+        iyy="${(m/12) * (w*w + d*d)}" iyz="0.0"
+        izz="${(m/12) * (w*w + h*h)}" />
     </inertial>
   </xacro:macro>
   <xacro:macro name="cylinder_inertia" params="m r h">
     <inertial>
-      <origin xyz="0 0 0" rpy="${pi1/2} 0 0" />
-      <mass value="${m}"/>
-      <inertia ixx="${(m/12) * (3*r*r + h*h)}" ixy = "0" ixz = "0" iyy="${(m/12) * (3*r*r + h*h)}" iyz = "0" izz="${(m/2) * (r*r)}"/>
+      <origin xyz="0 0 0" rpy="${pi/2} 0 0" />
+      <mass value="${m}" />
+      <inertia ixx="${(m/12) * (3*r*r + h*h)}" ixy="0" ixz="0"
+        iyy="${(m/12) * (3*r*r + h*h)}" iyz="0"
+        izz="${(m/2) * (r*r)}" />
     </inertial>
   </xacro:macro>
-  <!-- Wheel macro -->
-  <xacro:macro name="wheel" params="name width radius mass color">
+  <!-- Wheel Macro -->
+  <!--
+       The macro takes a wheel name and an offset (x,y,z) relative to the base_link.
+       Here, x_offset is chosen as half the wheel_base (front wheels: +, rear: -).
+       y_offset is half the wheel_track (left: positive, right: negative).
+       z_offset is set so that the wheel center is at the ground level (z = wheel_radius).
+  -->
+  <xacro:macro name="wheel" params="name x_offset y_offset z_offset is_right">
     <link name="${name}">
       <visual>
-        <origin xyz="0 0 0" rpy="${pi1/2} 0 0"/>
+        <!-- Rotate the cylinder so its axis (default along z) aligns with the desired rolling axis -->
+        <origin xyz="0 0 0" rpy="0 0 ${pi/2}" />
         <geometry>
-          <cylinder length="${width}" radius="${radius}"/>
+          <cylinder radius="${wheel_radius}" length="${wheel_thickness}" />
         </geometry>
-        <material name="${color}" />
+        <material name="black">
+          <color rgba="0 0 0 1" />
+        </material>
       </visual>
       <collision>
-        <origin xyz="0 0 0" rpy="${pi1/2} 0 0"/>
+        <origin xyz="0 0 0" rpy="0 1.5708 0" />
         <geometry>
-          <cylinder length="${width}" radius="${radius}"/>
+          <cylinder radius="${wheel_radius}" length="${wheel_thickness}" />
         </geometry>
       </collision>
-    <xacro:cylinder_inertia m="${mass}" r="${radius}" h="${width}"/>
+      <!-- Use cylinder_inertia for the wheel (mass = 1) -->
+      <xacro:cylinder_inertia m="1" r="${wheel_radius}" h="${wheel_thickness}" />
     </link>
+    <joint name="${name}_joint" type="continuous">
+      <parent link="base_link" />
+      <child link="${name}" />
+      <xacro:if value="${is_right}">
+        <origin xyz="${x_offset} ${y_offset} ${z_offset}" rpy="${pi/2} 0 0" />
+      </xacro:if>
+      <xacro:unless value="${is_right}">
+        <origin xyz="${x_offset} ${y_offset} ${z_offset}" rpy="${-pi/2} 0 ${0}" />
+      </xacro:unless>
+      <!-- Set the axis to align with the rolling direction; adjust if needed -->
+      <axis xyz="0 0 1" />
+      <limit effort="5.0" velocity="5.0" />
+    </joint>
   </xacro:macro>
 </robot>
