Commit message: Update robot model and visualization configuration for improved accuracy and clarity

File: vector_description/urdf/model.urdf.xacro (robot description, xacro)
@@ -1,23 +1,22 @@
 <?xml version="1.0"?>
-<robot xmlns:xacro="http://ros.org/wiki/xacro">
+<robot name="vector_robot" xmlns:xacro="http://ros.org/wiki/xacro">
     <!-- Xacro Properties -->
     <!-- TODO: Use correct dimensions -->
     <!-- Base dimensions -->
-    <xacro:property name="base_length" value="0.5" />         <!-- Length of the base -->
+    <xacro:property name="base_length" value="0.55" />         <!-- Length of the base -->
     <xacro:property name="base_width" value="0.3" />          <!-- Width of the base -->
     <xacro:property name="base_height" value="0.2" />         <!-- Height of the base -->
-    <xacro:property name="base_ground_clearance" value="0.1" /> <!-- Distance from ground to base
-    bottom -->
+    <xacro:property name="base_ground_clearance" value="0.2" /> <!-- Distance from ground to base bottom -->
     <!-- Wheel placement (symmetric) -->
-    <xacro:property name="wheel_base" value="0.4" />          <!-- Distance between front and back wheels -->
-    <xacro:property name="wheel_track" value="0.3" />         <!-- Distance between left and right wheels -->
+    <xacro:property name="wheel_base" value="0.6" />          <!-- Distance between front and back wheels -->
+    <xacro:property name="wheel_track" value="0.4" />         <!-- Distance between left and right wheels -->
     <!-- Wheel dimensions -->
-    <xacro:property name="wheel_radius" value="0.1" />
-    <xacro:property name="wheel_thickness" value="0.05" />
+    <xacro:property name="wheel_radius" value="0.254" />   <!-- 10 inches - 0.254 meters -->
+    <xacro:property name="wheel_thickness" value="0.0635" /> <!-- 2.5 inches - 0.0635 meters -->
     <!-- Base Link Definition -->
     <link name="base_link">
         <visual>
             <!-- Raise the base so its bottom is at ground clearance -->
-            <origin xyz="0 0 ${base_ground_clearance + base_height/2}" rpy="0 0 0" />
+            <origin xyz="0 0 0" rpy="0 0 0" />
             <geometry>
                 <box size="${base_length} ${base_width} ${base_height}" />
@@ -28,5 +27,5 @@
         </visual>
         <collision>
-            <origin xyz="0 0 ${base_ground_clearance + base_height/2}" rpy="0 0 0" />
+            <origin xyz="0 0 0" rpy="0 0 0" />
             <geometry>
                 <box size="${base_length} ${base_width} ${base_height}" />
@@ -36,15 +35,24 @@
         <xacro:box_inertia m="10" w="${base_width}" h="${base_height}" d="${base_length}" />
     </link>
+    <!-- Base Frame Link -->
+    <link name="base_footprint">
+        <visual>
+            <origin xyz="0 0 0" rpy="0 0 0" />
+        </visual>
+    </link>
+    <!-- Base Joint -->
+    <joint name="base_link_joint" type="fixed">
+        <parent link="base_footprint" />
+        <child link="base_link" />
+        <origin xyz="0 0 ${base_ground_clearance + base_height/2}" rpy="0 0 0" />
+    </joint>
     <!-- Instantiate Four Wheels -->
-    <!-- Front wheels: x_offset = +wheel_base/2, Rear wheels: x_offset = -wheel_base/2 -->
-    <!-- Left wheels: y_offset = +wheel_track/2, Right wheels: y_offset = -wheel_track/2 -->
-    <!-- z_offset is set to wheel_radius so that the wheel touches the ground -->
-    <xacro:wheel name="front_left_wheel" x_offset="${wheel_base/2}" y_offset="${wheel_track/2}"
-        z_offset="${wheel_radius}" is_right="false" />
-    <xacro:wheel name="front_right_wheel" x_offset="${wheel_base/2}" y_offset="${-wheel_track/2}"
-        z_offset="${wheel_radius}" is_right="true" />
-    <xacro:wheel name="rear_left_wheel" x_offset="${-wheel_base/2}" y_offset="${wheel_track/2}"
-        z_offset="${wheel_radius}" is_right="false" />
-    <xacro:wheel name="rear_right_wheel" x_offset="${-wheel_base/2}" y_offset="${-wheel_track/2}"
-        z_offset="${wheel_radius}" is_right="true" />
+    <xacro:wheel name="front_left_wheel" x_offset="${wheel_base/2}" y_offset="${wheel_track/2 + wheel_thickness/2}"
+        z_offset="${-base_ground_clearance }" is_right="false" />
+    <xacro:wheel name="front_right_wheel" x_offset="${wheel_base/2}" y_offset="${-(wheel_track/2 +  wheel_thickness/2)}"
+        z_offset="${-base_ground_clearance }" is_right="true" />
+    <xacro:wheel name="rear_left_wheel" x_offset="${-wheel_base/2}" y_offset="${wheel_track/2 + wheel_thickness/2}"
+        z_offset="${-base_ground_clearance }" is_right="false" />
+    <xacro:wheel name="rear_right_wheel" x_offset="${-wheel_base/2}" y_offset="${-(wheel_track/2 +  wheel_thickness/2)}"
+        z_offset="${-base_ground_clearance }" is_right="true" />
 </robot>

Commit message: Add vector_bringup package with launch and configuration files for robot bringup

File: vector_description/urdf/model.urdf.xacro (robot description, xacro)
@@ -18,11 +18,12 @@
         <visual>
             <!-- Raise the base so its bottom is at ground clearance -->
-            <origin xyz="0 0 0" rpy="0 0 0" />
+            <origin xyz="0 0 0" rpy="${-pi/2} 0 0" />
             <geometry>
-                <box size="${base_length} ${base_width} ${base_height}" />
+                <!-- <box size="${base_length} ${base_width} ${base_height}" /> -->
+                <mesh filename="package://vector_description/meshes/vector_base.dae" />
             </geometry>
-            <material name="blue">
+            <!-- <material name="blue">
                 <color rgba="0 0 1 1" />
-            </material>
+            </material> -->
         </visual>
         <collision>

File: vector_description/urdf/utils.urdf.xacro (robot description, xacro)
@@ -56,9 +56,10 @@
         <origin xyz="0 0 0" rpy="0 0 ${pi/2}" />
         <geometry>
-          <cylinder radius="${wheel_radius}" length="${wheel_thickness}" />
+          <!-- <cylinder radius="${wheel_radius}" length="${wheel_thickness}" /> -->
+            <mesh filename="package://vector_description/meshes/vector_wheel.dae" />
         </geometry>
-        <material name="black">
+        <!-- <material name="black">
           <color rgba="0 0 0 1" />
-        </material>
+        </material> -->
       </visual>
       <collision>

Commit message: Refactor URDF files and add Gazebo plugin configuration for improved robot simulation

File: vector_description/urdf/model.urdf.xacro (robot description, xacro)
@@ -1,4 +1,4 @@
 <?xml version="1.0"?>
-<robot name="vector_robot" xmlns:xacro="http://ros.org/wiki/xacro">
+<robot name="vector" xmlns:xacro="http://ros.org/wiki/xacro">
     <!-- Xacro Properties -->
     <!-- TODO: Use correct dimensions -->
@@ -12,5 +12,5 @@
     <xacro:property name="wheel_track" value="0.4" />         <!-- Distance between left and right wheels -->
     <!-- Wheel dimensions -->
-    <xacro:property name="wheel_radius" value="0.254" />   <!-- 10 inches - 0.254 meters -->
+    <xacro:property name="wheel_radius" value="0.127" />   <!-- 10 inches - 0.254 meters -->
     <xacro:property name="wheel_thickness" value="0.0635" /> <!-- 2.5 inches - 0.0635 meters -->
     <!-- Base Link Definition -->

File: vector_description/urdf/robot.urdf.xacro (robot description, xacro)
@@ -1,7 +1,10 @@
 <?xml version="1.0"?>
-<robot name="vector_robot" xmlns:xacro="http://ros.org/wiki/xacro">
+<robot name="vector"
+  xmlns:xacro="http://ros.org/wiki/xacro">
   <!-- Include utility macros and properties -->
   <xacro:include filename="$(find vector_description)/urdf/utils.urdf.xacro" />
   <!-- Include the model definition -->
   <xacro:include filename="$(find vector_description)/urdf/model.urdf.xacro" />
+  <!-- Include the gazebo plugins -->
+  <xacro:include filename="$(find vector_description)/urdf/gazebo.urdf.xacro" />
 </robot>

File: vector_description/urdf/utils.urdf.xacro (robot description, xacro)
@@ -64,5 +64,5 @@
       </visual>
       <collision>
-        <origin xyz="0 0 0" rpy="0 1.5708 0" />
+        <origin xyz="0 0 0" rpy="0 0 ${pi/2}" />
         <geometry>
           <cylinder radius="${wheel_radius}" length="${wheel_thickness}" />

Commit message: Implemented diff drive plugin for robot teleoperation in Gazebo and and fix some of the alignments of the components in the robot model.

File: vector_description/urdf/model.urdf.xacro (robot description, xacro)
@@ -9,9 +9,9 @@
     <xacro:property name="base_ground_clearance" value="0.2" /> <!-- Distance from ground to base bottom -->
     <!-- Wheel placement (symmetric) -->
-    <xacro:property name="wheel_base" value="0.6" />          <!-- Distance between front and back wheels -->
-    <xacro:property name="wheel_track" value="0.4" />         <!-- Distance between left and right wheels -->
+    <xacro:property name="wheel_base" value="0.53" />          <!-- Distance between front and back wheels -->
+    <xacro:property name="wheel_track" value="0.555" />         <!-- Distance between left and right wheels -->
     <!-- Wheel dimensions -->
     <xacro:property name="wheel_radius" value="0.127" />   <!-- 10 inches - 0.254 meters -->
-    <xacro:property name="wheel_thickness" value="0.0635" /> <!-- 2.5 inches - 0.0635 meters -->
+    <xacro:property name="wheel_thickness" value="0.05" /> <!-- 2.5 inches - 0.0635 meters -->
     <!-- Base Link Definition -->
     <link name="base_link">
@@ -34,5 +34,5 @@
         </collision>
         <!-- Use box_inertia macro for base_link (mass = 10) -->
-        <xacro:box_inertia m="10" w="${base_width}" h="${base_height}" d="${base_length}" />
+        <xacro:box_inertia m="1" w="${base_width}" h="${base_height}" d="${base_length}" />
     </link>
     <!-- Base Frame Link -->
@@ -40,4 +40,6 @@
         <visual>
             <origin xyz="0 0 0" rpy="0 0 0" />
+            <geometry>
+            </geometry>
         </visual>
     </link>
@@ -50,10 +52,10 @@
     <!-- Instantiate Four Wheels -->
     <xacro:wheel name="front_left_wheel" x_offset="${wheel_base/2}" y_offset="${wheel_track/2 + wheel_thickness/2}"
-        z_offset="${-base_ground_clearance }" is_right="false" />
+        z_offset="${-base_ground_clearance + 0.02 }" is_right="false" />
     <xacro:wheel name="front_right_wheel" x_offset="${wheel_base/2}" y_offset="${-(wheel_track/2 +  wheel_thickness/2)}"
-        z_offset="${-base_ground_clearance }" is_right="true" />
+        z_offset="${-base_ground_clearance + 0.02 }" is_right="true" />
     <xacro:wheel name="rear_left_wheel" x_offset="${-wheel_base/2}" y_offset="${wheel_track/2 + wheel_thickness/2}"
-        z_offset="${-base_ground_clearance }" is_right="false" />
+        z_offset="${-base_ground_clearance + 0.02 }" is_right="false" />
     <xacro:wheel name="rear_right_wheel" x_offset="${-wheel_base/2}" y_offset="${-(wheel_track/2 +  wheel_thickness/2)}"
-        z_offset="${-base_ground_clearance }" is_right="true" />
+        z_offset="${-base_ground_clearance + 0.02 }" is_right="true" />
 </robot>

File: vector_description/urdf/sensors/diff_drive.xacro (robot description, xacro)
@@ -42,7 +42,7 @@
       <max_linear_velocity>2.0</max_linear_velocity>
       <!-- Sets the minimum angular velocity. Overrides <min_velocity> if set. -->
-      <min_angular_velocity>-1.0</min_angular_velocity>
+      <min_angular_velocity>-5.0</min_angular_velocity>
       <!-- Sets the maximum angular velocity. Overrides <max_velocity> if set. -->
-      <max_angular_velocity>1.0</max_angular_velocity>
+      <max_angular_velocity>5.0</max_angular_velocity>
       <!-- Sets the minimum linear acceleration. Overrides <min_acceleration> if set. -->
       <!-- <min_linear_acceleration>0.0</min_linear_acceleration> -->

File: vector_description/urdf/utils.urdf.xacro (robot description, xacro)
@@ -29,7 +29,5 @@
       <origin xyz="0 0 0" rpy="${pi/2} 0 ${pi/2}" />
       <mass value="${m}" />
-      <inertia ixx="${(m/12) * (h*h + d*d)}" ixy="0.0" ixz="0.0"
-        iyy="${(m/12) * (w*w + d*d)}" iyz="0.0"
-        izz="${(m/12) * (w*w + h*h)}" />
+      <inertia ixx="${(m/12) * (h*h + d*d)}" ixy="0.0" ixz="0.0" iyy="${(m/12) * (w*w + d*d)}" iyz="0.0" izz="${(m/12) * (w*w + h*h)}" />
     </inertial>
   </xacro:macro>
@@ -38,7 +36,5 @@
       <origin xyz="0 0 0" rpy="${pi/2} 0 0" />
       <mass value="${m}" />
-      <inertia ixx="${(m/12) * (3*r*r + h*h)}" ixy="0" ixz="0"
-        iyy="${(m/12) * (3*r*r + h*h)}" iyz="0"
-        izz="${(m/2) * (r*r)}" />
+      <inertia ixx="${(m/12) * (3*r*r + h*h)}" ixy="0" ixz="0" iyy="${(m/12) * (3*r*r + h*h)}" iyz="0" izz="${(m/2) * (r*r)}" />
     </inertial>
   </xacro:macro>
@@ -54,8 +50,8 @@
       <visual>
         <!-- Rotate the cylinder so its axis (default along z) aligns with the desired rolling axis -->
-        <origin xyz="0 0 0" rpy="0 0 ${pi/2}" />
+        <origin xyz="0 0 0" rpy="${pi} 0 ${pi/2}" />
         <geometry>
           <!-- <cylinder radius="${wheel_radius}" length="${wheel_thickness}" /> -->
-            <mesh filename="package://vector_description/meshes/vector_wheel.dae" />
+          <mesh filename="package://vector_description/meshes/vector_wheel.dae" />
         </geometry>
         <!-- <material name="black">
@@ -64,11 +60,19 @@
       </visual>
       <collision>
-        <origin xyz="0 0 0" rpy="0 0 ${pi/2}" />
+        <origin xyz="0 0 -0.023" rpy="0 0 ${pi/2}" />
         <geometry>
           <cylinder radius="${wheel_radius}" length="${wheel_thickness}" />
         </geometry>
+        <surface>
+          <friction>
+            <ode>
+              <mu>0.8</mu>
+              <mu2>0.8</mu2>
+            </ode>
+          </friction>
+        </surface>
       </collision>
-      <!-- Use cylinder_inertia for the wheel (mass = 1) -->
-      <xacro:cylinder_inertia m="1" r="${wheel_radius}" h="${wheel_thickness}" />
+      <!-- Use cylinder_inertia for the wheel (mass = 1.15) -->
+      <xacro:cylinder_inertia m="0.3" r="${wheel_radius}" h="${wheel_thickness}" />
     </link>
     <joint name="${name}_joint" type="continuous">
@@ -77,11 +81,12 @@
       <xacro:if value="${is_right}">
         <origin xyz="${x_offset} ${y_offset} ${z_offset}" rpy="${pi/2} 0 0" />
+        <axis xyz="0 0 -1" />
       </xacro:if>
       <xacro:unless value="${is_right}">
         <origin xyz="${x_offset} ${y_offset} ${z_offset}" rpy="${-pi/2} 0 ${0}" />
+        <axis xyz="0 0 1" />
       </xacro:unless>
-      <!-- Set the axis to align with the rolling direction; adjust if needed -->
-      <axis xyz="0 0 1" />
-      <limit effort="5.0" velocity="5.0" />
+      <limit effort="1.0" velocity="1000000000"/>
+      <dynamics damping="0.00000000000000000001" friction="0.0000000001"/>
     </joint>
   </xacro:macro>
