Commit message: Add sensor configurations and launch arguments for improved robot simulation

File: vector_description/urdf/gazebo.urdf.xacro (robot description, xacro)
@@ -3,11 +3,14 @@
     xmlns:xacro="http://www.ros.org/wiki/xacro">
     <!-- ........................... INCLUDE PLUGINS ................................... -->
-    <!-- <xacro:include filename="$(find vector_description)/urdf/sensors/rgbd_camera.xacro" /> -->
-    <!-- <xacro:include filename="$(find vector_description)/urdf/sensors/battery.xacro" /> -->
+    <xacro:if value="$(arg camera_enabled)">
+        <xacro:include filename="$(find vector_description)/urdf/sensors/rgbd_camera.xacro" />
+    </xacro:if>
+    <xacro:if value="$(arg two_d_lidar_enabled)">
+        <xacro:include filename="$(find vector_description)/urdf/sensors/lidar.xacro" />
+    </xacro:if>
+    <xacro:include filename="$(find vector_description)/urdf/sensors/battery.xacro" />
     <xacro:include filename="$(find vector_description)/urdf/sensors/diff_drive.xacro" />
-    <!-- <xacro:include filename="$(find vector_description)/urdf/sensors/lidar.xacro" /> -->
-    <!-- <xacro:include filename="$(find vector_description)/urdf/sensors/imu.xacro" /> -->
-s
-        <!-- ........................... SENSOR PLUGIN ................................... -->
+    <xacro:include filename="$(find vector_description)/urdf/sensors/imu.xacro" />
+    <!-- ........................... SENSOR PLUGIN ................................... -->
     <gazebo>
         <plugin filename="ignition-gazebo-sensors-system" name="ignition::gazebo::systems::Sensors">

File: vector_description/urdf/robot.urdf.xacro (robot description, xacro)
@@ -2,4 +2,11 @@
 <robot name="vector"
   xmlns:xacro="http://ros.org/wiki/xacro">
+  <!-- Xacro Arguments -->
+  <xacro:arg name="wheel_odom_topic" default="odometry/filtered"/>
+  <xacro:arg name="camera_enabled" default="false"/>
+  <xacro:arg name="two_d_lidar_enabled" default="false"/>
+  <xacro:arg name="ground_truth_odometry" default="false"/>
+  <xacro:arg name="is_simulation" default="true"/>
+  <!-- <xacro:property name="odom_topic" value="$(arg wheel_odom_topic)"/> -->
   <!-- Include utility macros and properties -->
   <xacro:include filename="$(find vector_description)/urdf/utils.urdf.xacro" />
@@ -7,4 +14,6 @@
   <xacro:include filename="$(find vector_description)/urdf/model.urdf.xacro" />
   <!-- Include the gazebo plugins -->
-  <xacro:include filename="$(find vector_description)/urdf/gazebo.urdf.xacro" />
+  <xacro:if value="$(arg is_simulation)">
+    <xacro:include filename="$(find vector_description)/urdf/gazebo.urdf.xacro" />
+  </xacro:if>
 </robot>

File: vector_description/urdf/sensors/diff_drive.xacro (robot description, xacro)
@@ -9,55 +9,33 @@
       <right_joint>front_right_wheel_joint</right_joint>
       <right_joint>rear_right_wheel_joint</right_joint>
-      <!-- Distance between wheels, in meters. The default value is 1.0m. -->
-      <wheel_separation>0.4</wheel_separation>
-      <!-- Wheel radius in meters. The default value is 0.2m. -->
-      <wheel_radius>0.127</wheel_radius>
-      <!-- Odometry publication frequency. This element is optional, and the default value is 50Hz. -->
-      <odom_publish_frequency>30</odom_publish_frequency>
-      <!-- Custom topic that this system will subscribe to in order to receive command velocity messages. This element is optional, and the default value is /model/{name_of_model}/cmd_vel. -->
-      <topic>/cmd_vel</topic>
-      <!-- Custom topic on which this system will publish odometry messages. This element is optional, and the default value is /model/{name_of_model}/odometry. -->
-      <odom_topic>/odometry/filtered</odom_topic>
-      <!-- Custom topic on which this system will publish the transform from frame_id to child_frame_id. This element is optional, and the default value is /model/{name_of_model}/tf. -->
-      <tf_topic>/tf</tf_topic>
-      <!-- Custom frame_id field that this system will use as the origin of the odometry transform in both the <tf_topic> gz.msgs.Pose_V message and the <odom_topic> gz.msgs.Odometry message. This element is optional, and the default value is {name_of_model}/odom. -->
-      <frame_id>odom</frame_id>
-      <!-- Custom child_frame_id that this system will use as the target of the odometry transform in both the <tf_topic> gz.msgs.Pose_V message and the <odom_topic> gz.msgs.Odometry message. This element is optional, and the default value is {name_of_model}/{name_of_link}. -->
-      <child_frame_id>base_link</child_frame_id>
-      <!-- Sets both the minimum linear and minimum angular velocity. -->
+      <wheel_separation>0.4</wheel_separation>      <!-- Distance between wheels, in meters. The default value is 1.0m. -->
+      <wheel_radius>0.127</wheel_radius>      <!-- Wheel radius in meters. The default value is 0.2m. -->
+      <odom_publish_frequency>30</odom_publish_frequency>      <!-- Odometry publication frequency. This element is optional, and the default value is 50Hz. -->
+      <topic>/cmd_vel</topic>      <!-- Custom topic that this system will subscribe to in order to receive command velocity messages. This element is optional, and the default value is /model/{name_of_model}/cmd_vel. -->
+      <xacro:unless value="$(arg ground_truth_odometry)">
+        <odom_topic>$(arg wheel_odom_topic)</odom_topic>        <!-- Custom topic on which this system will publish odometry messages. This element is optional, and the default value is /model/{name_of_model}/odometry. -->
+        <tf_topic>/tf</tf_topic>        <!-- Custom topic on which this system will publish the transform from frame_id to child_frame_id. This element is optional, and the default value is /model/{name_of_model}/tf. -->
+      </xacro:unless>
+      <frame_id>odom</frame_id>      <!-- Custom frame_id field that this system will use as the origin of the odometry transform in both the <tf_topic> gz.msgs.Pose_V message and the <odom_topic> gz.msgs.Odometry message. This element is optional, and the default value is {name_of_model}/odom. -->
+      <child_frame_id>base_link</child_frame_id>      <!-- Custom child_frame_id that this system will use as the target of the odometry transform in both the <tf_topic> gz.msgs.Pose_V message and the <odom_topic> gz.msgs.Odometry message. This element is optional, and the default value is {name_of_model}/{name_of_link}. -->
       <!-- <min_velocity>0.0</min_velocity> -->
-      <!-- Sets both the maximum linear and maximum angular velocity. -->
       <!-- <max_velocity>2.0</max_velocity> -->
-      <!-- Sets both the minimum linear and minimum angular acceleration. -->
       <!-- <min_acceleration>0.0</min_acceleration> -->
-      <!-- Sets both the maximum linear and maximum angular acceleration. -->
       <!-- <max_acceleration>1.0</max_acceleration> -->
-      <!-- Sets both the minimum linear and minimum angular jerk. -->
       <!-- <min_jerk>0.0</min_jerk> -->
-      <!-- Sets both the maximum linear and maximum angular jerk. -->
       <!-- <max_jerk>1.0</max_jerk> -->
       <!-- Sets the minimum linear velocity. Overrides <min_velocity> if set. -->
       <min_linear_velocity>-2.0</min_linear_velocity>
-      <!-- Sets the maximum linear velocity. Overrides <max_velocity> if set. -->
       <max_linear_velocity>2.0</max_linear_velocity>
-      <!-- Sets the minimum angular velocity. Overrides <min_velocity> if set. -->
       <min_angular_velocity>-5.0</min_angular_velocity>
-      <!-- Sets the maximum angular velocity. Overrides <max_velocity> if set. -->
       <max_angular_velocity>5.0</max_angular_velocity>
       <!-- Sets the minimum linear acceleration. Overrides <min_acceleration> if set. -->
       <!-- <min_linear_acceleration>0.0</min_linear_acceleration> -->
-      <!-- Sets the maximum linear acceleration. Overrides <max_acceleration> if set. -->
       <!-- <max_linear_acceleration>0.2</max_linear_acceleration> -->
-      <!-- Sets the minimum angular acceleration. Overrides <min_acceleration> if set. -->
       <!-- <min_angular_acceleration>0.0</min_angular_acceleration> -->
-      <!-- Sets the maximum angular acceleration. Overrides <max_acceleration> if set. -->
       <!-- <max_angular_acceleration>1.0</max_angular_acceleration> -->
-      <!-- Sets the minimum linear jerk. Overrides <min_jerk> if set. -->
       <!-- <min_linear_jerk>0.0</min_linear_jerk> -->
-      <!-- Sets the maximum linear jerk. Overrides <max_jerk> if set. -->
       <!-- <max_linear_jerk>0.5</max_linear_jerk> -->
-      <!-- Sets the minimum angular jerk. Overrides <min_jerk> if set. -->
       <!-- <min_angular_jerk>0.0</min_angular_jerk> -->
-      <!-- Sets the maximum angular jerk. Overrides <max_jerk> if set. -->
       <!-- <max_angular_jerk>0.5</max_angular_jerk> -->
     </plugin>
@@ -65,13 +43,15 @@
   <!-- ............................. ground truth .................................... -->
   <!-- Second method to get odometry-->
-  <!-- <gazebo>
-    <plugin filename="libignition-gazebo6-odometry-publisher-system" name="ignition::gazebo::systems::OdometryPublisher">
-      <odom_frame>odom</odom_frame>
-      <robot_base_frame>base_link</robot_base_frame>
-      <odom_topic>/odom/filtered</odom_topic>
-      <tf_topic>/tf</tf_topic>
-      <dimensions>2</dimensions>
-      <odom_publish_frequency>10</odom_publish_frequency>
-    </plugin>
-  </gazebo> -->
+  <xacro:if value="$(arg ground_truth_odometry)">
+    <gazebo>
+      <plugin filename="libignition-gazebo6-odometry-publisher-system" name="ignition::gazebo::systems::OdometryPublisher">
+        <odom_frame>odom</odom_frame>
+        <robot_base_frame>base_link</robot_base_frame>
+        <odom_topic>$(arg wheel_odom_topic)</odom_topic>
+        <tf_topic>/tf</tf_topic>
+        <dimensions>2</dimensions>
+        <odom_publish_frequency>10</odom_publish_frequency>
+      </plugin>
+    </gazebo>
+  </xacro:if>
 </robot>

Commit message: Update sensor positions and launch configurations for improved robot functionality

File: vector_description/urdf/gazebo.urdf.xacro (robot description, xacro)
@@ -9,5 +9,5 @@
         <xacro:include filename="$(find vector_description)/urdf/sensors/lidar.xacro" />
     </xacro:if>
-    <xacro:include filename="$(find vector_description)/urdf/sensors/battery.xacro" />
+    <!-- <xacro:include filename="$(find vector_description)/urdf/sensors/battery.xacro" /> -->
     <xacro:include filename="$(find vector_description)/urdf/sensors/diff_drive.xacro" />
     <xacro:include filename="$(find vector_description)/urdf/sensors/imu.xacro" />

File: vector_description/urdf/model.urdf.xacro (robot description, xacro)
@@ -36,17 +36,12 @@
         <xacro:box_inertia m="1" w="${base_width}" h="${base_height}" d="${base_length}" />
     </link>
-    <!-- Base Frame Link -->
+    <!-- Base Footprint Link -->
     <link name="base_footprint">
-        <visual>
-            <origin xyz="0 0 0" rpy="0 0 0" />
-            <geometry>
-            </geometry>
-        </visual>
     </link>
-    <!-- Base Joint -->
+    <!-- Base Footprint Joint -->
     <joint name="base_link_joint" type="fixed">
-        <parent link="base_footprint" />
-        <child link="base_link" />
-        <origin xyz="0 0 ${base_ground_clearance + base_height/2}" rpy="0 0 0" />
+        <parent link="base_link" />
+        <child link="base_footprint" />
+        <origin xyz="0 0 ${-(base_ground_clearance + base_height/2)}" rpy="0 0 0" />
     </joint>
     <!-- Instantiate Four Wheels -->

File: vector_description/urdf/sensors/lidar.xacro (robot description, xacro)
@@ -25,5 +25,5 @@
         <parent link="base_link"/>
         <child link="laser"/>
-        <origin xyz="0 0 ${(base_height/2 + 0.005)}" rpy="0 0 0"/>
+        <origin xyz="0 0 ${(base_height/2 + 0.05)}" rpy="0 0 0"/>
     </joint>
     <!-- Lidar Sensor -->

File: vector_description/urdf/sensors/rgbd_camera.xacro (robot description, xacro)
@@ -25,5 +25,5 @@
         <parent link="base_link"/>
         <child link="camera_link"/>
-        <origin xyz="0 0 ${(base_length/2 + 0.005)}" rpy="0 0 0"/>
+        <origin xyz="${(base_length/2 + 0.005)} 0 ${(base_height/2 + 0.05)}" rpy="0 0 0"/>
     </joint>
     <!-- RGBD Camera Sensor -->
